File: hardware/pcb/eagle/spool_tmc2130_b.sch (EAGLE design)
At the start: 29 parts, among them J1 PINHD-1X8, J2 F-1X08-SIP-100-40, J3 F-1X02-SIP-100-32, K1 G6K-2P-Y, U1 NJM7805SDL, U2 ATTINY85-20PU, X1 JST-XH-02-PIN-LONG-PAD, X2 JST-XH-04-PIN-LONG-PAD, X3 JST-XH-02-PIN-LONG-PAD, X4 JST-XH-02-PIN-LONG-PAD, X5 JST-XH-02-PIN-LONG-PAD, X6 JST-XH-02-PIN-LONG-PAD, X9 JST-XH-03-PIN-LONG-PAD

Commit message: Control board rev.B: EAGLE files, schematic PDF, BOM and docs
The board was revised in Autodesk Fusion and exported in EAGLE 9.7.0
format. rev.A (as built) is kept in tag pcb-rev.A.

- EXT_SENSE: X5 pin 2 and JP2 pin 1 to ATtiny85 PB4 through R6 10k,
  pull-down R5 10k
- T1 DTC123JKA, R2 2.2k, D3 driven from Pro Mini D8 with R4 470
- Chip resistors 0603 -> 0805
- Schematic and board netlists identical (26 nets); connectivity of
  all nets checked on the Gerber output of the CAM processor
- Schematic PDF (A3) added
- BOM, wiring, README, LICENSE (Autodesk Resistor library) and
  CHANGELOG updated

Co-Authored-By: Claude Opus 5.5 <noreply@anthropic.com>
Claude-Session: https://claude.ai/code/session_01CN5z7kNkBV6zKj8DLApdnx
Parts:
- added R5, R6: 10k, Resistor:R-US_CHIP-0805(2012-METRIC)
- C1: value (none) -> 100uF
- C2: value RDER73A103K2K1H03B -> 0.33uF
- C3: value RDER73A103K2K1H03B -> 0.1uF
- PS1: value (none) -> RXEF135
- R1, R3: device resistor:R-US_R0603 -> Resistor:R-US_CHIP-0805(2012-METRIC)
- R2: value 680 -> 2.2k; device resistor:R-US_R0603 -> Resistor:R-US_CHIP-0805(2012-METRIC)
- R4: value 150 -> 470; device resistor:R-US_R0603 -> Resistor:R-US_CHIP-0805(2012-METRIC)
- T1: value (none) -> DTC123JKA
Connections:
- new net D8_LED: ARDUINO1.D8, D3.A
- new net EXT_SENSE: JP2.1, R5.2, R6.1, X5-2.S
- new net N$1: R6.2, U2.PB4
- net D4: no longer D3.A
- net EXT_IN: no longer JP2.1, X5-2.S
- net GND: now also R5.1
